File: eagle/clock.sch (EAGLE design)
At the start: 0 parts

Commit message: .
Parts:
- added C1: (no value), rcl:C-EUC0805
- added C2: 10mF, rcl:CPOL-EUA/3216-18W
- added C3: 100mF, rcl:CPOL-EUA/3216-18W
- added IC1: LM1117MPX-3.3, lm1117:LM1117MPX-3.3
- added JP1: (no value), pinhead:PINHD-2X4
- added JP2: (no value), pinhead:PINHD-1X5
- added PH1: D1160_12, photo-elements:D1160_12
- added R1: (no value), rcl:R-EU_M0805
- added U$1: MICRO-USB, microusb:MICRO-USB
- added U2: (no value), esp8266modules:ESP12ESMD
Connections:
- new net +3V3: C3.+, IC1.OUT, IC1.OUT1, U2.VCC
- new net +5V: C2.+, IC1.IN, U$1.VCC
- new net GND: C2.-, C3.-, IC1.GND, U$1.GND, U$1.GND@1, U$1.GND@2, U2.GND
