File: eagle/clock.sch (EAGLE design)
At the start: 10 parts, among them IC1 LM1117MPX-3.3

Commit message: .
Parts:
- added G1: CH291-1220LF, battery:CH291-1220LF
- added R2, R3, R4, R5, R6: (no value), rcl:R-EU_M0805
- added U$2: DS3231, DS3231:DS3231
- JP1: value (none) -> PROG
- JP2: value (none) -> DISPLAY
Connections:
- new net CH_PD: JP1.3, R5.1, U2.CH_PD
- new net DSP_CLK: JP2.2
- new net DSP_CS: JP2.3
- new net DSP_DIN: JP2.1
- new net LIGHT_SENSOR: C1.1, PH1.2, R3.2, U2.ADC
- new net N$1: G1.+, U$2.VBAT
- new net N$2: R6.1, U2.GPIO15
- new net N$3: U$2.VCC
- new net RESET: JP1.5, R4.1, U$2.RST, U2.RESET
- new net RX: JP1.8, U2.RX
- new net SCL: R2.1, U$2.SCL
- new net SDA: R1.1, U$2.SDA
- new net SQW: U$2.32KHZ
- new net TIMER_INT: U$2.INT
- new net TX: JP1.1, U2.TX
- net +3V3: now also PH1.1, R1.2, R2.2, R4.2, R5.2
- net +5V: now also JP2.5
- net GND: now also C1.2, G1.-, JP1.2, JP2.4, R3.1, R6.2, U$2.GND, U$2.P$1, U$2.P$2, U$2.P$3, U$2.P$4, U$2.P$5, U$2.P$6, U$2.P$7, U$2.P$8
Other:
- moved on the sheet: C1, JP1, JP2, PH1, R1, U2

Commit message: First version of board design
Parts:
- added C4, C5: 100u, rcl:C-EUC0805
- added LED1: G, led:LEDCHIPLED_0805
- added R7: 4.7k, rcl:R-EU_M0805
- added R8: 330, rcl:R-EU_M0805
- added U$3: BMP085, bmp085:BMP085
- C1: value (none) -> 100u
- R1, R2, R4, R5, R6: value (none) -> 4.7k
- R3: value (none) -> 68k
- U2: value (none) -> ESP12E
Connections:
- net N$1 renamed VBAT
- net N$2 renamed GPIO15
- net +3V3: now also C4.1, C5.1, JP1.7, R7.2, R8.2, U$2.VCC, U$3.VDDA, U$3.VDDD
- net DSP_CLK: now also U2.GPIO14
- net DSP_CS: now also U2.GPIO2
- net DSP_DIN: now also U2.GPIO13
- net GND: now also C4.2, C5.2, LED1.C, U$3.GND
- net N$3: now also LED1.A, R8.1; no longer U$2.VCC
- net SCL: now also U$3.SCL, U2.GPIO5
- net SDA: now also U$3.SDA, U2.GPIO4
- net TIMER_INT: now also R7.1, U2.GPIO12
Other:
- moved on the sheet: C1, G1, JP1, JP2, PH1, R1, R2, R3, R4, R5, R6, U2

Commit message: board updated
Connections:
- new net GPIO0: JP1.6, U2.GPIO0
- new net N$2: U2.GPIO16
Changed lines of the file:
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@@
+</segment>
+</net>
+<net name="GPIO0" class="0">
+<segment>
+<pinref part="U2" gate="G$1" pin="GPIO0"/>
+<wire x1="144.78" y1="15.24" x2="152.4" y2="15.24" width="0.1524" layer="91"/>
+<label x="152.4" y="15.24" size="1.27" layer="95" xref="yes"/>
+</segment>
+<segment>
+<pinref part="JP1" gate="A" pin="6"/>
+<wire x1="27.94" y1="-17.78" x2="35.56" y2="-17.78" width="0.1524" layer="91"/>
+<label x="35.56" y="-17.78" size="1.27" layer="95" xref="yes"/>
+</segment>
+</net>
+<net name="N$2" class="0">
+<segment>
+<pinref part="U2" gate="G$1" pin="GPIO16"/>
+<wire x1="111.76" y1="17.78" x2="104.14" y2="17.78" width="0.1524" layer="91"/>
+<label x="104.14" y="17.78" size="1.27" layer="95" rot="MR0" xref="yes"/>
 </segment>
 </net>

Commit message: final design
Parts:
- removed U$3: BMP085, bmp085:BMP085
- added JP3: I2C, pinhead:PINHD-1X4
- added U1: BMP180, bmp180:BMP180
Connections:
- removed net N$2: U2.GPIO16
- new net GPIO2: JP1.4, U2.GPIO2
- net +3V3: now also JP3.3, U1.VDD, U1.VDDIO; no longer U$3.VDDA, U$3.VDDD
- net DSP_CS: now also U2.GPIO16; no longer U2.GPIO2
- net GND: now also JP3.4, U1.GND; no longer U$3.GND
- net SCL: now also JP3.1, U1.SCL; no longer U$3.SCL
- net SDA: now also JP3.2, U1.SDA; no longer U$3.SDA
Other:
- moved on the sheet: R1, R2, R4, R5, R7

Commit message: .
Parts:
- removed PH1: D1160_12, photo-elements:D1160_12
- removed U1: BMP180, bmp180:BMP180
- added IC2: DS3231, DS3231_industrialberry:DS3231SOIC-16W
- U$2: value DS3231 -> GL5537; device DS3231:DS3231 -> misc:GL5537
Connections:
- removed net VBAT: G1.+, U$2.VBAT
- new net N$4: G1.+, IC2.VBAT
- net +3V3: now also IC2.VCC, U$2.P$2; no longer PH1.1, R8.2, U$2.VCC, U1.VDD, U1.VDDIO
- net +5V: now also R8.2
- net GND: now also IC2.GND, IC2.NC@1, IC2.NC@2, IC2.NC@3, IC2.NC@4, IC2.NC@5, IC2.NC@6, IC2.NC@7, IC2.NC@8; no longer U$2.GND, U$2.P$1, U$2.P$2, U$2.P$3, U$2.P$4, U$2.P$5, U$2.P$6, U$2.P$7, U$2.P$8, U1.GND
- net LIGHT_SENSOR: now also U$2.P$1; no longer PH1.2
- net RESET: now also IC2.!RST; no longer U$2.RST
- net SCL: now also IC2.SCL; no longer U$2.SCL, U1.SCL
- net SDA: now also IC2.SDA; no longer U$2.SDA, U1.SDA
- net SQW: now also IC2.32KHZ; no longer U$2.32KHZ
- net TIMER_INT: now also IC2.!INT; no longer U$2.INT
Other:
- moved on the sheet: G1, LED1, R8
