File: eagle/clock.brd (EAGLE design)
At the start: 100 x 80 mm, 0 parts

Commit message: .
Parts:
- added C1: (no value), rcl:C0805
- added C2: 10mF, rcl:A/3216-18W
- added C3: 100mF, rcl:A/3216-18W
- added IC1: LM1117MPX-3.3, lm1117:SOT223
- added JP1: (no value), pinhead:2X04
- added JP2: (no value), pinhead:1X05
- added PH1: D1160_12, photo-elements:D11XX
- added R1: (no value), rcl:M0805
- added U$1: MICRO-USB, microusb:MICRO-USB
- added U2: (no value), esp8266modules:ESP12E-SMD
Connections:
- new net +3V3: C3.+, IC1.2, IC1.TAB, U2.VCC
- new net +5V: C2.+, IC1.3, U$1.1
- new net GND: C2.-, C3.-, IC1.1, U$1.5, U$1.GND1, U$1.GND2, U2.GND
Other:
- board size 100 x 80 mm -> 74 x 33 mm

Commit message: .
Parts:
- added G1: CH291-1220LF, battery:CH291-1220LF
- added R2, R3, R4, R5, R6: (no value), rcl:M0805
- added U$2: DS3231, DS3231:SO16
- JP1: value (none) -> PROG
- JP2: value (none) -> DISPLAY
- moved JP2 49.0 mm to (88.3, 28.4)
- moved C2 38.3 mm to (13.0, 19.0)
- moved JP1 36.4 mm to (86.4, 16.4)
- moved C3 30.0 mm to (21.0, 38.0)
- moved IC1 28.3 mm to (13.0, 12.0), turned to 90 degrees
Connections:
- new net CH_PD: JP1.3, R5.1, U2.CH_PD
- new net DSP_CLK: JP2.2
- new net DSP_CS: JP2.3
- new net DSP_DIN: JP2.1
- new net LIGHT_SENSOR: C1.1, PH1.2, R3.2, U2.ADC
- new net N$1: G1.+, U$2.14
- new net N$2: R6.1, U2.GPIO15
- new net N$3: U$2.2
- new net RESET: JP1.5, R4.1, U$2.4, U2.RESET
- new net RX: JP1.8, U2.RXD0
- new net SCL: R2.1, U$2.16
- new net SDA: R1.1, U$2.15
- new net SQW: U$2.1
- new net TIMER_INT: U$2.3
- new net TX: JP1.1, U2.TXD0
- net +3V3: now also PH1.1, R1.2, R2.2, R4.2, R5.2
- net +5V: now also JP2.5
- net GND: now also C1.2, G1.-, JP1.2, JP2.4, R3.1, R6.2, U$2.10, U$2.11, U$2.12, U$2.13, U$2.5, U$2.6, U$2.7, U$2.8, U$2.9

Commit message: First version of board design
Parts:
- added C4, C5: 100u, rcl:C0805
- added LED1: G, led:CHIPLED_0805
- added R7: 4.7k, rcl:M0805
- added R8: 330, rcl:M0805
- added U$3: BMP085, bmp085:BMP085
- C1: value (none) -> 100u
- R1, R2, R4, R5, R6: value (none) -> 4.7k
- R3: value (none) -> 68k
- U2: value (none) -> ESP12E
- moved R3 77.4 mm to (20.0, 27.0)
- moved R4 66.9 mm to (20.0, 30.0), turned to 180 degrees
- moved JP1 65.7 mm to (21.9, 3.85)
- moved R6 63.3 mm to (49.5, 13.5)
- moved R2 50.6 mm to (49.5, 19.5)
- moved U$2 46.4 mm to (53.0, 6.50), turned to 180 degrees
- moved G1 43.8 mm to (61.0, 14.0)
- moved R5 39.6 mm to (20.0, 21.0), turned to 180 degrees
- moved C3 35.2 mm to (12.0, 4.00), turned to 180 degrees
- moved U2 26.0 mm to (34.8, 17.4)
- moved R1 24.1 mm to (49.5, 16.5)
- moved JP2 20.3 mm to (72.3, 15.8), turned to 270 degrees
- moved PH1 17.9 mm to (11.7, 26.8), turned to 270 degrees
- moved C1 4.61 mm to (20.0, 23.9), turned to 180 degrees
- moved C2 3.16 mm to (12.0, 16.0), turned to 180 degrees
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Connections:
- net N$1 renamed VBAT
- net N$2 renamed GPIO15
- net +3V3: now also C4.1, C5.1, JP1.7, R7.2, R8.2, U$2.2, U$3.3, U$3.4
- net DSP_CLK: now also U2.GPIO14
- net DSP_CS: now also U2.GPIO2
- net DSP_DIN: now also U2.GPIO13
- net GND: now also C4.2, C5.2, LED1.C, U$3.1
- net N$3: now also LED1.A, R8.1; no longer U$2.2
- net SCL: now also U$3.6, U2.GPIO5
- net SDA: now also U$3.7, U2.GPIO4
- net TIMER_INT: now also R7.1, U2.GPIO12
Routing:
- net +3V3: track 0.00 -> 135.9 mm, vias 0 -> 2
- net +5V: track 0.00 -> 93.7 mm
- net RESET: track 0.00 -> 65.8 mm, vias 0 -> 2
- net DSP_CLK: track 0.00 -> 64.1 mm, vias 0 -> 2
- net DSP_DIN: track 0.00 -> 54.0 mm
- net TIMER_INT: track 0.00 -> 43.7 mm
- net SCL: track 0.00 -> 40.7 mm
- net DSP_CS: track 0.00 -> 35.4 mm, vias 0 -> 2
- net TX: track 0.00 -> 34.6 mm, vias 0 -> 2
- net SDA: track 0.00 -> 33.6 mm, vias 0 -> 3
- net RX: track 0.00 -> 24.5 mm, vias 0 -> 1
- net CH_PD: track 0.00 -> 24.4 mm, vias 0 -> 1
- net LIGHT_SENSOR: track 0.00 -> 19.6 mm
- net VBAT: track 0.00 -> 11.8 mm
- net GPIO15: track 0.00 -> 6.56 mm
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- added copper zone on layer 1, net GND
- added copper zone on layer 16, net GND
Other:
- board size 74 x 33 mm -> 75 x 32 mm

Commit message: board updated
Connections:
- new net GPIO0: JP1.6, U2.GPIO0
- new net N$2: U2.GPIO16
Routing:
- net GPIO0: track 0.00 -> 23.9 mm
- net DSP_DIN: track 54.0 -> 68.1 mm
- net DSP_CLK: track 64.1 -> 50.2 mm
- net SCL: track 40.7 -> 46.2 mm
- net RESET: track 65.8 -> 70.5 mm, vias 2 -> 1
- net TIMER_INT: track 43.7 -> 48.1 mm, vias 0 -> 2
- net SDA: track 33.6 -> 36.6 mm
- net +5V: track 93.7 -> 96.0 mm
- net RX: track 24.5 -> 25.2 mm
- net CH_PD: track 24.4 -> 23.9 mm
