File: eagle/clock.brd (EAGLE design)
At the start: 75 x 32 mm, 23 parts, among them IC1 LM1117MPX-3.3, U2 ESP12E

Commit message: final design
Parts:
- removed U$3: BMP085, bmp085:BMP085
- added JP3: I2C, pinhead:1X04
- added U1: BMP180, bmp180:BMP180
- moved LED1 20.2 mm to (3.50, 23.7), turned to 270 degrees
- moved R8 17.5 mm to (3.50, 21.0), turned to 0 degrees
- moved C5 5.50 mm to (20.0, 14.5), turned to 0 degrees
- moved C4 2.50 mm to (44.0, 2.50), turned to 180 degrees
- moved U$2 1.12 mm to (52.0, 6.00), turned to 0 degrees
- moved R7 0.44 mm to (20.0, 17.6)
- moved R5 0.33 mm to (20.0, 20.7)
- moved JP1 0.22 mm to (21.7, 3.75)
- moved C1 0.17 mm to (20.0, 23.8)
- moved R3 0.11 mm to (20.0, 26.9)
Connections:
- removed net N$2: U2.GPIO16
- new net GPIO2: JP1.4, U2.GPIO2
- net +3V3: now also JP3.3, U1.2, U1.3; no longer U$3.3, U$3.4
- net DSP_CS: now also U2.GPIO16; no longer U2.GPIO2
- net GND: now also JP3.4, U1.7; no longer U$3.1
- net SCL: now also JP3.1, U1.5; no longer U$3.6
- net SDA: now also JP3.2, U1.6; no longer U$3.7
Routing:
- net GPIO2: track 0.00 -> 34.2 mm
- net +3V3: track 136.3 -> 166.5 mm, vias 2 -> 3
- net SDA: track 36.6 -> 60.1 mm
- net DSP_DIN: track 68.1 -> 49.9 mm, vias 0 -> 1
- net DSP_CS: track 35.2 -> 49.6 mm
- net RESET: track 70.5 -> 59.7 mm, vias 1 -> 2
- net +5V: track 96.0 -> 85.5 mm, vias 0 -> 2
- net TIMER_INT: track 48.1 -> 38.4 mm, vias 2 -> 4
- net RX: track 25.2 -> 32.7 mm, vias 1 -> 0
- net TX: track 34.9 -> 38.5 mm, vias 2 -> 1
- net DSP_CLK: track 50.2 -> 47.1 mm, vias 2 -> 1
- net GPIO0: track 23.9 -> 26.1 mm
- net CH_PD: track 23.9 -> 25.7 mm, vias 1 -> 0
- net VBAT: track 11.8 -> 13.4 mm
- net SCL: track 46.2 -> 47.3 mm
Other:
- board text added: "Clock board v2"

Commit message: .
Parts:
- removed PH1: D1160_12, photo-elements:D11XX
- removed U1: BMP180, bmp180:BMP180
- added IC2: DS3231, DS3231_industrialberry:SOIC-16W
- U$2: value DS3231 -> GL5537; device DS3231:SO16 -> misc:GL55
- moved U$2 44.5 mm to (13.0, 27.5), turned to 90 degrees
- moved JP3 13.0 mm to (47.0, 3.00)
- moved R2 11.7 mm to (47.5, 8.00), turned to 270 degrees
- moved G1 11.7 mm to (53.0, 22.5), turned to 270 degrees
- moved C4 11.0 mm to (53.5, 8.00), turned to 90 degrees
- moved R1 8.56 mm to (50.5, 8.00), turned to 270 degrees
- moved R6 2.24 mm to (48.5, 11.5)
- turned C2 to 0 degrees
- turned C3 to 0 degrees
- turned C5 to 180 degrees
Connections:
- removed net VBAT: G1.+, U$2.14
- new net N$4: G1.+, IC2.14
- net +3V3: now also IC2.2, U$2.P$2; no longer PH1.1, R8.2, U$2.2, U1.2, U1.3
- net +5V: now also R8.2
- net GND: now also IC2.10, IC2.11, IC2.12, IC2.13, IC2.5, IC2.6, IC2.7, IC2.8, IC2.9; no longer U$2.10, U$2.11, U$2.12, U$2.13, U$2.5, U$2.6, U$2.7, U$2.8, U$2.9, U1.7
- net LIGHT_SENSOR: now also U$2.P$1; no longer PH1.2
- net RESET: now also IC2.4; no longer U$2.4
- net SCL: now also IC2.16; no longer U$2.16, U1.5
- net SDA: now also IC2.15; no longer U$2.15, U1.6
- net SQW: now also IC2.1; no longer U$2.1
- net TIMER_INT: now also IC2.3; no longer U$2.3
Routing:
- net +3V3: track 166.5 -> 102.0 mm, vias 3 -> 0
- net SDA: track 60.1 -> 30.8 mm, vias 3 -> 1
- net TIMER_INT: track 38.4 -> 63.1 mm, vias 4 -> 2
- net SCL: track 47.3 -> 30.8 mm, vias 0 -> 2
- net RESET: track 59.7 -> 74.9 mm, vias 2 -> 1
- net N$4: track 0.00 -> 14.1 mm
- net VBAT: track 13.4 -> 0.00 mm
- net +5V: track 85.5 -> 78.0 mm, vias 2 -> 1
- net RX: track 32.7 -> 25.6 mm, vias 0 -> 1
- net DSP_DIN: track 49.9 -> 56.6 mm
- net TX: track 38.5 -> 44.2 mm
- net CH_PD: track 25.7 -> 29.5 mm, vias 0 -> 1
- net DSP_CLK: track 47.1 -> 49.9 mm
- net DSP_CS: track 49.6 -> 47.2 mm, vias 2 -> 1
- net GPIO15: track 6.60 -> 4.89 mm
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Other:
- board text removed: "Clock board v2"
