File: eagle/driver.brd (EAGLE design)
At the start: 80 x 35 mm, 4 parts

Commit message: max7219 connection
Parts:
- added C1, C2, C3, C4: (no value), rcl:C0805
- added R1, R2, R3, R4: (no value), rcl:R0805
- added U$2, U$3, U$4, U$5: MAX7219CWG, max7219:SO24L
- added U$6: BMP085, bmp085:BMP085
- added U1: BMP180, bmp180:BMP180
Connections:
- new net M1C1: U$1.P$64, U$2.2
- new net M1C2: U$1.P$63, U$2.11
- new net M1C3: U$1.P$62, U$2.6
- new net M1C4: U$1.P$61, U$2.7
- new net M1C5: U$1.P$60, U$2.3
- new net M1C6: U$1.P$59, U$2.10
- new net M1C7: U$1.P$58, U$2.5
- new net M1C8: U$1.P$57, U$2.8
- new net M1R1: U$1.P$1, U$2.14
- new net M1R2: U$1.P$2, U$2.16
- new net M1R3: U$1.P$3, U$2.20
- new net M1R4: U$1.P$4, U$2.23
- new net M1R5: U$1.P$5, U$2.21
- new net M1R6: U$1.P$6, U$2.15
- new net M1R7: U$1.P$7, U$2.17
- new net M1R8: U$1.P$8, U$2.22
- new net M2C1: U$1.P$56, U$3.2
- new net M2C2: U$1.P$55, U$3.11
- new net M2C3: U$1.P$54, U$3.6
- new net M2C4: U$1.P$53, U$3.7
- new net M2C5: U$1.P$52, U$3.3
- new net M2C6: U$1.P$51, U$3.10
- new net M2C7: U$1.P$50, U$3.5
- new net M2C8: U$1.P$49, U$3.8
- new net M2R1: U$1.P$9, U$3.14
- new net M2R2: U$1.P$10, U$3.16
- new net M2R3: U$1.P$11, U$3.20
- new net M2R4: U$1.P$12, U$3.23
- new net M2R5: U$1.P$13, U$3.21
- new net M2R6: U$1.P$14, U$3.15
- new net M2R7: U$1.P$15, U$3.17
- new net M2R8: U$1.P$16, U$3.22
- new net M3C1: U$1.P$48, U$4.2
- new net M3C2: U$1.P$47, U$4.11
- new net M3C3: U$1.P$46, U$4.6
- new net M3C4: U$1.P$45, U$4.7
- new net M3C5: U$1.P$44, U$4.3
- new net M3C6: U$1.P$43, U$4.10
- new net M3C7: U$1.P$42, U$4.5
- new net M3C8: U$1.P$41, U$4.8
- new net M3R1: U$1.P$17, U$4.14
- new net M3R2: U$1.P$18, U$4.16
- new net M3R3: U$1.P$19, U$4.20
- new net M3R4: U$1.P$20, U$4.23
- new net M3R5: U$1.P$21, U$4.21
- new net M3R6: U$1.P$22, U$4.15
- new net M3R7: U$1.P$23, U$4.17
- new net M3R8: U$1.P$24, U$4.22
- new net M4C1: U$1.P$40, U$5.2
- new net M4C2: U$1.P$39, U$5.11
- new net M4C3: U$1.P$38, U$5.6
- new net M4C4: U$1.P$37, U$5.7
- new net M4C5: U$1.P$36, U$5.3
- new net M4C6: U$1.P$35, U$5.10
- new net M4C7: U$1.P$34, U$5.5
- new net M4C8: U$1.P$33, U$5.8
- new net M4R1: U$1.P$25, U$5.14
- new net M4R2: U$1.P$26, U$5.16
- new net M4R3: U$1.P$27, U$5.20
- new net M4R4: U$1.P$28, U$5.23
- new net M4R5: U$1.P$29, U$5.21
- new net M4R6: U$1.P$30, U$5.15
- new net M4R7: U$1.P$31, U$5.17
- new net M4R8: U$1.P$32, U$5.22
- new net N$10: R2.2, U$3.18
- new net N$13: U$3.24, U$4.1
- new net N$15: R3.2, U$4.18
- new net N$18: U$4.24, U$5.1
- new net N$19: U$5.24
- new net N$20: R4.2, U$5.18
- new net N$5: R1.2, U$2.18
- new net N$8: U$2.24, U$3.1
- net +3V3: now also U$6.3, U$6.4, U1.2, U1.3
- net +5V: now also C1.1, C2.1, C3.1, C4.1, R1.1, R2.1, R3.1, R4.1, U$2.19, U$3.19, U$4.19, U$5.19
- net DSP_CLK: now also U$2.13, U$3.13, U$4.13, U$5.13
- net DSP_CS: now also U$2.12, U$3.12, U$4.12, U$5.12
- net DSP_DIN: now also U$2.1
- net GND: now also C1.2, C2.2, C3.2, C4.2, U$1.GND@1, U$1.GND@2, U$1.GND@3, U$1.GND@4, U$2.4, U$2.9, U$3.4, U$3.9, U$4.4, U$4.9, U$5.4, U$5.9, U$6.1, U1.7
- net SCL: now also U$6.6, U1.5
- net SDA: now also U$6.7, U1.6
